File: Hardware/Qwiic 1x1/BMP384 Breakout.sch (EAGLE design)
At the start: 25 parts, among them J1 QWIIC_RIGHT_ANGLE, J2 QWIIC_RIGHT_ANGLE, U1 BMP384

Commit message: Remove library file
BMP384 is in SFE Eagle library, update part in design
Parts:
- U1: device bmp384:BMP384 -> SparkFun-Sensors:BMP384
Changed lines of the file:
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@@
 <parts>
 <part name="FRAME1" library="SparkFun-Aesthetics" deviceset="FRAME-LETTER" device=""/>
-<part name="U1" library="bmp384" deviceset="BMP384" device=""/>
+<part name="U1" library="SparkFun-Sensors" deviceset="BMP384" device=""/>
 <part name="GND1" library="SparkFun-PowerSymbols" deviceset="GND" device=""/>
 <part name="SUPPLY1" library="SparkFun-PowerSymbols" deviceset="VDD" device=""/>
